File: kicad/board_trace/board_trace.kicad_pcb (KiCad board)
At the start: 2 copper layers, 40.7 x 62.4 mm, 61 parts, among them J1 USB3 stacked Type-A (candidat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, J2 USB3 stacked Type-A (candidat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, J3 SFP20 (candidate), J4 DC barrel jack (unidentified), U1 VL813 (candidate), U2 UNKNOWN, Y1 25MHz

Commit message: board_trace: place CND-tek C5441174 SFP+ 1x1 cage, fit to connector J3
Add C5441174 (MPN 201N1Y02001) cage footprint: 17 plated legs (7x 1.05 + 9x 0.95 + 1x 0.85 mm) on two rows 14.25 mm apart plus a 3-hole end row. Its land matches the board's 17 cage holes exactly.

Place CAGE1 at (158.4663, 111.2747) rotation 0 - centred on J3 X, +12.0 mm toward the module end; connector J3 unchanged.

Keep superseded C42931382 footprint (mis-labelled QSFP-derived import with 3 bogus pads) for history; add cage_fit.svg/pdf exports. Also commit pending 2026-09-13 HANDOFF.md and design/STATUS.md updates.
Parts:
- added CAGE1: C5441174_CAGE-SFP-1X1-TH, lcsc:C5441174_CAGE-SFP-1X1-TH, F.Cu at (158.5, 111.3)
