File: kicad/usb3_sfp_hub/hub_support.kicad_sch (KiCad schematic)
At the start: 32 parts, among them J7 5.0-5.2V at board / input TBD, J9 Short 1-2 to request reset / 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, U12 TPS3808G33DBVR, Y1 25MHz / CL and package TBD

Commit message: usb3_sfp_hub: source JLCPCB parts; 3x3mm filter inductors and damping resistor
L1/L2: replace the unavailable Coilcraft XGL4020-472MEC (LCSC stock 1) with cjiang FTC303018D4R7MBCA (LCSC C5832388), 3x3mm matching the calipered reference board, on Inductor_SMD:L_Changjiang_FTC303020D.

R1/R2: replace the untraceable Panasonic ERJ8RQFR43V (no LCSC listing) with FH RTF06KR430FTG (LCSC C44453441), same 0.43 ohm 1% 1206 current-sense damping.

- Assign LCSC/JLCPCB numbers to the settled passives and ICs; export to bom.csv.
- Rebase check_sfp_power_budget on the real 72mOhm filter DCR and report the 0.10 ohm allocation gap instead of asserting it away.
- Regenerate the six sheets, netlist, budget JSON, BOM and previews; update README and sfp_filter_evidence.json.
- Drop stale analyzer dumps (bom/analysis.json, validation/schematic_analysis.json) and ignore the regenerated copies.

Connectivity check PASS (105 components). ERC and full analog/optical qualification remain open; no PCB.
Parts:
- C20, C21, C22, C23, C24, C25, C26, C27, C28, C29, C30, C31, C32, C33, C34, C35, C38: LCSC (none) -> C1525; MPN (none) -> CL05B104KO5NNNC; Manufacturer (none) -> Samsung Electro-Mechanics
- R24: LCSC (none) -> C25804; MPN (none) -> 0603WAF1002T5E; Manufacturer (none) -> UNI-ROYAL
- R9: LCSC (none) -> C22864; MPN (none) -> 0603WAF1212T5E; Manufacturer (none) -> UNI-ROYAL
- U12: LCSC (none) -> C43698
