File: kicad/usb3_sfp_hub/port_power.kicad_sch (KiCad schematic)
At the start: 30 parts, among them U2 TPS2553DBVR, U3 TPS2553DBVR, U4 TPS2553DBVR, U5 TPS2553DBVR, U6 SN74LVC1G04DBVR

Commit message: usb3_sfp_hub: source JLCPCB parts; 3x3mm filter inductors and damping resistor
L1/L2: replace the unavailable Coilcraft XGL4020-472MEC (LCSC stock 1) with cjiang FTC303018D4R7MBCA (LCSC C5832388), 3x3mm matching the calipered reference board, on Inductor_SMD:L_Changjiang_FTC303020D.

R1/R2: replace the untraceable Panasonic ERJ8RQFR43V (no LCSC listing) with FH RTF06KR430FTG (LCSC C44453441), same 0.43 ohm 1% 1206 current-sense damping.

- Assign LCSC/JLCPCB numbers to the settled passives and ICs; export to bom.csv.
- Rebase check_sfp_power_budget on the real 72mOhm filter DCR and report the 0.10 ohm allocation gap instead of asserting it away.
- Regenerate the six sheets, netlist, budget JSON, BOM and previews; update README and sfp_filter_evidence.json.
- Drop stale analyzer dumps (bom/analysis.json, validation/schematic_analysis.json) and ignore the regenerated copies.

Connectivity check PASS (105 components). ERC and full analog/optical qualification remain open; no PCB.
Parts:
- C39, C41, C42, C44, C45, C47, C48, C50, C51: LCSC (none) -> C1525; MPN (none) -> CL05B104KO5NNNC; Manufacturer (none) -> Samsung Electro-Mechanics
- R10, R11, R12, R13: LCSC (none) -> C2930078; MPN (none) -> FRC0603F2322TS; Manufacturer (none) -> FOJAN
- R14, R15, R16, R17: LCSC (none) -> C25804; MPN (none) -> 0603WAF1002T5E; Manufacturer (none) -> UNI-ROYAL
- R18, R19, R20, R21: LCSC (none) -> C21190; MPN (none) -> 0603WAF1001T5E; Manufacturer (none) -> UNI-ROYAL
- U2, U3, U4, U5: LCSC (none) -> C55266
- U6: LCSC (none) -> C7827
