File: kicad/usb3_sfp_hub/sfp_support.kicad_sch (KiCad schematic)
At the start: 16 parts, among them J6 3.3V management access / foot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

Commit message: usb3_sfp_hub: source JLCPCB parts; 3x3mm filter inductors and damping resistor
L1/L2: replace the unavailable Coilcraft XGL4020-472MEC (LCSC stock 1) with cjiang FTC303018D4R7MBCA (LCSC C5832388), 3x3mm matching the calipered reference board, on Inductor_SMD:L_Changjiang_FTC303020D.

R1/R2: replace the untraceable Panasonic ERJ8RQFR43V (no LCSC listing) with FH RTF06KR430FTG (LCSC C44453441), same 0.43 ohm 1% 1206 current-sense damping.

- Assign LCSC/JLCPCB numbers to the settled passives and ICs; export to bom.csv.
- Rebase check_sfp_power_budget on the real 72mOhm filter DCR and report the 0.10 ohm allocation gap instead of asserting it away.
- Regenerate the six sheets, netlist, budget JSON, BOM and previews; update README and sfp_filter_evidence.json.
- Drop stale analyzer dumps (bom/analysis.json, validation/schematic_analysis.json) and ignore the regenerated copies.

Connectivity check PASS (105 components). ERC and full analog/optical qualification remain open; no PCB.
Parts:
- C10, C13: LCSC (none) -> C21397
- C11, C12, C14, C9: LCSC (none) -> C1525; MPN (none) -> CL05B104KO5NNNC; Manufacturer (none) -> Samsung Electro-Mechanics
- L1, L2: value 4.7uH / XGL4020-472MEC -> 4.7uH / FTC303018D4R7MBCA; footprint power:L_Coilcraft_XGL4020 -> Inductor_SMD:L_Changjiang_FTC303020D; BOM Comments 47.3mOhm max DCR at 25C; 1.9/3.0/4.1A Isat at 10/20/30% dro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 -> 3x3mm molded, sized to the calipered reference board; 72mOh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; LCSC (none) -> C5832388; MPN XGL4020-472MEC -> FTC303018D4R7MBCA; Manufacturer Coilcraft -> Changjiang (cjiang)
- R1, R2: BOM Comments 1206 damping candidate; nominal total R about 0.494Ohm at 1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 -> 430mOhm 1% 250mW current-sense, 1206; nominal total R about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; LCSC (none) -> C44453441; MPN ERJ8RQFR43V -> RTF06KR430FTG; Manufacturer Panasonic -> FH
- R3, R4, R5, R6, R7: LCSC (none) -> C23162; MPN (none) -> 0603WAF4701T5E; Manufacturer (none) -> UNI-ROYAL
