File: kicad/usb3_sfp_hub/usb3_esd.kicad_sch (KiCad schematic)
At the start: 4 parts, among them U10 TPD4E02B04DQAR, U11 TPD4E02B04DQAR, U8 TPD4E02B04DQAR, U9 TPD4E02B04DQAR

Commit message: usb3_sfp_hub: source JLCPCB parts; 3x3mm filter inductors and damping resistor
L1/L2: replace the unavailable Coilcraft XGL4020-472MEC (LCSC stock 1) with cjiang FTC303018D4R7MBCA (LCSC C5832388), 3x3mm matching the calipered reference board, on Inductor_SMD:L_Changjiang_FTC303020D.

R1/R2: replace the untraceable Panasonic ERJ8RQFR43V (no LCSC listing) with FH RTF06KR430FTG (LCSC C44453441), same 0.43 ohm 1% 1206 current-sense damping.

- Assign LCSC/JLCPCB numbers to the settled passives and ICs; export to bom.csv.
- Rebase check_sfp_power_budget on the real 72mOhm filter DCR and report the 0.10 ohm allocation gap instead of asserting it away.
- Regenerate the six sheets, netlist, budget JSON, BOM and previews; update README and sfp_filter_evidence.json.
- Drop stale analyzer dumps (bom/analysis.json, validation/schematic_analysis.json) and ignore the regenerated copies.

Connectivity check PASS (105 components). ERC and full analog/optical qualification remain open; no PCB.
Parts:
- U10, U11, U8, U9: LCSC (none) -> C106794
Changed lines of the file:
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@@
 (property "Placement target" "J2 SuperSpeed contacts; TX connector side of AC capacitors; short ground returns at pins 3/8" (at 99.06 63.5 0) (effects (font (size 1 1)) hide))
 (property "BOM Comments" "Bidirectional +/-3.6V signal-only TVS; 0.25pF typical, 0.33pF max at 0V/1MHz/25C. NC pads used for PCB flow-through, not internally connected. SI/ESD tests pending." (at 99.06 63.5 0) (effects (font (size 1 1)) hide))
+(property "LCSC" "C106794" (at 99.06 63.5 0) (effects (font (size 1 1)) hide))
 (pin "1")
 (pin "2")
@@
 (property "Placement target" "J3 SuperSpeed contacts; TX connector side of AC capacitors; short ground returns at pins 3/8" (at 299.72 63.5 0) (effects (font (size 1 1)) hide))
 (property "BOM Comments" "Bidirectional +/-3.6V signal-only TVS; 0.25pF typical, 0.33pF max at 0V/1MHz/25C. NC pads used for PCB flow-through, not internally connected. SI/ESD tests pending." (at 299.72 63.5 0) (effects (font (size 1 1)) hide))
+(property "LCSC" "C106794" (at 299.72 63.5 0) (effects (font (size 1 1)) hide))
 (pin "1")
 (pin "2")
@@
 (property "Placement target" "J4 SuperSpeed contacts; TX connector side of AC capacitors; short ground returns at pins 3/8" (at 99.06 137.16 0) (effects (font (size 1 1)) hide))
 (property "BOM Comments" "Bidirectional +/-3.6V signal-only TVS; 0.25pF typical, 0.33pF max at 0V/1MHz/25C. NC pads used for PCB flow-through, not internally connected. SI/ESD tests pending." (at 99.06 137.16 0) (effects (font (size 1 1)) hide))
+(property "LCSC" "C106794" (at 99.06 137.16 0) (effects (font (size 1 1)) hide))
 (pin "1")
 (pin "2")
@@
 (property "Placement target" "J5 SuperSpeed contacts; TX connector side of AC capacitors; short ground returns at pins 3/8" (at 299.72 137.16 0) (effects (font (size 1 1)) hide))
 (property "BOM Comments" "Bidirectional +/-3.6V signal-only TVS; 0.25pF typical, 0.33pF max at 0V/1MHz/25C. NC pads used for PCB flow-through, not internally connected. SI/ESD tests pending." (at 299.72 137.16 0) (effects (font (size 1 1)) hide))
+(property "LCSC" "C106794" (at 299.72 137.16 0) (effects (font (size 1 1)) hide))
 (pin "1")
 (pin "2")
