File: kicad/usb3_sfp_hub/usb3_sfp_hub.kicad_sch (KiCad schematic)
At the start: 14 parts, among them J1 SFP+ / MODULE TBD, J2 USB3-A PORT 1, J3 USB3-A PORT 2, J4 USB3-A PORT 3, J5 USB3-A PORT 4, U1 VL813(A1)

Commit message: usb3_sfp_hub: source JLCPCB parts; 3x3mm filter inductors and damping resistor
L1/L2: replace the unavailable Coilcraft XGL4020-472MEC (LCSC stock 1) with cjiang FTC303018D4R7MBCA (LCSC C5832388), 3x3mm matching the calipered reference board, on Inductor_SMD:L_Changjiang_FTC303020D.

R1/R2: replace the untraceable Panasonic ERJ8RQFR43V (no LCSC listing) with FH RTF06KR430FTG (LCSC C44453441), same 0.43 ohm 1% 1206 current-sense damping.

- Assign LCSC/JLCPCB numbers to the settled passives and ICs; export to bom.csv.
- Rebase check_sfp_power_budget on the real 72mOhm filter DCR and report the 0.10 ohm allocation gap instead of asserting it away.
- Regenerate the six sheets, netlist, budget JSON, BOM and previews; update README and sfp_filter_evidence.json.
- Drop stale analyzer dumps (bom/analysis.json, validation/schematic_analysis.json) and ignore the regenerated copies.

Connectivity check PASS (105 components). ERC and full analog/optical qualification remain open; no PCB.
Parts:
- C1, C2, C3, C4, C5, C6, C7, C8: LCSC (none) -> C1525; MPN (none) -> CL05B104KO5NNNC; Manufacturer (none) -> Samsung Electro-Mechanics
- U1: BOM Comments EOL reference baseline; footprint and operating circuit qualification pending -> EOL reference baseline; footprint and operating circuit qualification pending; no LCSC listing (VIA EOL)
Changed lines of the file:
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@@
 (property "Manufacturer" "VIA Labs" (at 170.18 50.8 0) (effects (font (size 1 1)) hide))
 (property "Datasheet" "../../VL813.pdf" (at 170.18 50.8 0) (effects (font (size 1 1)) hide))
-(property "BOM Comments" "EOL reference baseline; footprint and operating circuit qualification pending" (at 170.18 50.8 0) (effects (font (size 1 1)) hide))
+(property "BOM Comments" "EOL reference baseline; footprint and operating circuit qualification pending; no LCSC listing (VIA EOL)" (at 170.18 50.8 0) (effects (font (size 1 1)) hide))
 (pin "23")
 (pin "22")
@@
 (property "Manufacturer" "VIA Labs" (at 254 48.26 0) (effects (font (size 1 1)) hide))
 (property "Datasheet" "../../VL813.pdf" (at 254 48.26 0) (effects (font (size 1 1)) hide))
-(property "BOM Comments" "EOL reference baseline; footprint and operating circuit qualification pending" (at 254 48.26 0) (effects (font (size 1 1)) hide))
+(property "BOM Comments" "EOL reference baseline; footprint and operating circuit qualification pending; no LCSC listing (VIA EOL)" (at 254 48.26 0) (effects (font (size 1 1)) hide))
 (pin "59")
 (pin "60")
@@
 (property "Manufacturer" "VIA Labs" (at 254 91.44 0) (effects (font (size 1 1)) hide))
 (property "Datasheet" "../../VL813.pdf" (at 254 91.44 0) (effects (font (size 1 1)) hide))
-(property "BOM Comments" "EOL reference baseline; footprint and operating circuit qualification pending" (at 254 91.44 0) (effects (font (size 1 1)) hide))
+(property "BOM Comments" "EOL reference baseline; footprint and operating circuit qualification pending; no LCSC listing (VIA EOL)" (at 254 91.44 0) (effects (font (size 1 1)) hide))
 (pin "66")
 (pin "67")
@@
 (property "Manufacturer" "VIA Labs" (at 254 134.62 0) (effects (font (size 1 1)) hide))
 (property "Datasheet" "../../VL813.pdf" (at 254 134.62 0) (effects (font (size 1 1)) hide))
-(property "BOM Comments" "EOL reference baseline; footprint and operating circuit qualification pending" (at 254 134.62 0) (effects (font (size 1 1)) hide))
+(property "BOM Comments" "EOL reference baseline; footprint and operating circuit qualification pending; no LCSC listing (VIA EOL)" (at 254 134.62 0) (effects (font (size 1 1)) hide))
 (pin "3")
 (pin "4")
@@
 (property "Manufacturer" "VIA Labs" (at 254 177.8 0) (effects (font (size 1 1)) hide))
 (property "Datasheet" "../../VL813.pdf" (at 254 177.8 0) (effects (font (size 1 1)) hide))
-(property "BOM Comments" "EOL reference baseline; footprint and operating circuit qualification pending" (at 254 177.8 0) (effects (font (size 1 1)) hide))
+(property "BOM Comments" "EOL reference baseline; footprint and operating circuit qualification pending; no LCSC listing (VIA EOL)" (at 254 177.8 0) (effects (font (size 1 1)) hide))
 (pin "11")
 (pin "12")
@@
 (property "Manufacturer" "VIA Labs" (at 294.64 243.84 0) (effects (font (size 1 1)) hide))
 (property "Datasheet" "../../VL813.pdf" (at 294.64 243.84 0) (effects (font (size 1 1)) hide))
-(property "BOM Comments" "EOL reference baseline; footprint and operating circuit qualification pending" (at 294.64 243.84 0) (effects (font (size 1 1)) hide))
+(property "BOM Comments" "EOL reference baseline; footprint and operating circuit qualification pending; no LCSC listing (VIA EOL)" (at 294.64 243.84 0) (effects (font (size 1 1)) hide))
 (pin "9")
 (pin "10")
@@
 (property "Manufacturer" "VIA Labs" (at 60.96 215.9 0) (effects (font (size 1 1)) hide))
 (property "Datasheet" "../../VL813.pdf" (at 60.96 215.9 0) (effects (font (size 1 1)) hide))
-(property "BOM Comments" "EOL reference baseline; footprint and operating circuit qualification pending" (at 60.96 215.9 0) (effects (font (size 1 1)) hide))
+(property "BOM Comments" "EOL reference baseline; footprint and operating circuit qualification pending; no LCSC listing (VIA EOL)" (at 60.96 215.9 0) (effects (font (size 1 1)) hide))
 (pin "2")
 (pin "5")
@@
 (property "Manufacturer" "VIA Labs" (at 167.64 147.32 0) (effects (font (size 1 1)) hide))
 (property "Datasheet" "../../VL813.pdf" (at 167.64 147.32 0) (effects (font (size 1 1)) hide))
-(property "BOM Comments" "EOL reference baseline; footprint and operating circuit qualification pending" (at 167.64 147.32 0) (effects (font (size 1 1)) hide))
+(property "BOM Comments" "EOL reference baseline; footprint and operating circuit qualification pending; no LCSC listing (VIA EOL)" (at 167.64 147.32 0) (effects (font (size 1 1)) hide))
 (pin "1")
 (pin "21")
@@
 (property "Value" "100nF / 0402" (at 297.18 45.72 0) (effects (font (size 1 1))))
 (property "Footprint" "Capacitor_SMD:C_0402_1005Metric" (at 297.18 43.18 0) (effects (font (size 1 1)) hide))
+(property "LCSC" "C1525" (at 297.18 43.18 0) (effects (font (size 1 1)) hide))
+(property "MPN" "CL05B104KO5NNNC" (at 297.18 43.18 0) (effects (font (size 1 1)) hide))
+(property "Manufacturer" "Samsung Electro-Mechanics" (at 297.18 43.18 0) (effects (font (size 1 1)) hide))
 (pin "1")
 (pin "2")
@@
 (property "Value" "100nF / 0402" (at 297.18 55.88 0) (effects (font (size 1 1))))
 (property "Footprint" "Capacitor_SMD:C_0402_1005Metric" (at 297.18 53.34 0) (effects (font (size 1 1)) hide))
+(property "LCSC" "C1525" (at 297.18 53.34 0) (effects (font (size 1 1)) hide))
+(property "MPN" "CL05B104KO5NNNC" (at 297.18 53.34 0) (effects (font (size 1 1)) hide))
+(property "Manufacturer" "Samsung Electro-Mechanics" (at 297.18 53.34 0) (effects (font (size 1 1)) hide))
 (pin "1")
 (pin "2")
@@
 (property "Value" "100nF / 0402" (at 297.18 88.9 0) (effects (font (size 1 1))))
 (property "Footprint" "Capacitor_SMD:C_0402_1005Metric" (at 297.18 86.36 0) (effects (font (size 1 1)) hide))
+(property "LCSC" "C1525" (at 297.18 86.36 0) (effects (font (size 1 1)) hide))
+(property "MPN" "CL05B104KO5NNNC" (at 297.18 86.36 0) (effects (font (size 1 1)) hide))
+(property "Manufacturer" "Samsung Electro-Mechanics" (at 297.18 86.36 0) (effects (font (size 1 1)) hide))
 (pin "1")
 (pin "2")
@@
 (property "Value" "100nF / 0402" (at 297.18 99.06 0) (effects (font (size 1 1))))
 (property "Footprint" "Capacitor_SMD:C_0402_1005Metric" (at 297.18 96.52 0) (effects (font (size 1 1)) hide))
+(property "LCSC" "C1525" (at 297.18 96.52 0) (effects (font (size 1 1)) hide))
+(property "MPN" "CL05B104KO5NNNC" (at 297.18 96.52 0) (effects (font (size 1 1)) hide))
+(property "Manufacturer" "Samsung Electro-Mechanics" (at 297.18 96.52 0) (effects (font (size 1 1)) hide))
 (pin "1")
 (pin "2")
@@
 (property "Value" "100nF / 0402" (at 297.18 132.07999999999998 0) (effects (font (size 1 1))))
 (property "Footprint" "Capacitor_SMD:C_0402_1005Metric" (at 297.18 129.54 0) (effects (font (size 1 1)) hide))
+(property "LCSC" "C1525" (at 297.18 129.54 0) (effects (font (size 1 1)) hide))
+(property "MPN" "CL05B104KO5NNNC" (at 297.18 129.54 0) (effects (font (size 1 1)) hide))
+(property "Manufacturer" "Samsung Electro-Mechanics" (at 297.18 129.54 0) (effects (font (size 1 1)) hide))
 (pin "1")
 (pin "2")
@@
 (property "Value" "100nF / 0402" (at 297.18 142.23999999999998 0) (effects (font (size 1 1))))
 (property "Footprint" "Capacitor_SMD:C_0402_1005Metric" (at 297.18 139.7 0) (effects (font (size 1 1)) hide))
+(property "LCSC" "C1525" (at 297.18 139.7 0) (effects (font (size 1 1)) hide))
+(property "MPN" "CL05B104KO5NNNC" (at 297.18 139.7 0) (effects (font (size 1 1)) hide))
+(property "Manufacturer" "Samsung Electro-Mechanics" (at 297.18 139.7 0) (effects (font (size 1 1)) hide))
 (pin "1")
 (pin "2")
@@
 (property "Value" "100nF / 0402" (at 297.18 175.26 0) (effects (font (size 1 1))))
 (property "Footprint" "Capacitor_SMD:C_0402_1005Metric" (at 297.18 172.72 0) (effects (font (size 1 1)) hide))
+(property "LCSC" "C1525" (at 297.18 172.72 0) (effects (font (size 1 1)) hide))
+(property "MPN" "CL05B104KO5NNNC" (at 297.18 172.72 0) (effects (font (size 1 1)) hide))
+(property "Manufacturer" "Samsung Electro-Mechanics" (at 297.18 172.72 0) (effects (font (size 1 1)) hide))
 (pin "1")
 (pin "2")
@@
 (property "Value" "100nF / 0402" (at 297.18 185.42 0) (effects (font (size 1 1))))
 (property "Footprint" "Capacitor_SMD:C_0402_1005Metric" (at 297.18 182.88 0) (effects (font (size 1 1)) hide))
-(pin "1")
-(pin "2")
+(property "LCSC" "C1525" (at 297.18 182.88 0) (effects (font (size 1 1)) hide))
+(property "MPN" "CL05B104KO5NNNC" (at 297.18 182.88 0) (effects (font (size 1 1)) hide))
+(property "Manufacturer" "Samsung Electro-Mechanics" (at 297.18 182.88 0) (effects (font (size 1 1)) hide))
+(pin "1")
+(pin "2")

Commit message: usb3_sfp_hub: note GL3510-OSY52 as non-drop-in VL813 alternative
Record Genesys Logic GL3510-OSY52 (LCSC C7501408) against U1 and in the README as a non-drop-in replacement for the EOL VL813: QFN-64 USB3.1 Gen1 4-port with built-in 5V->3.3V/1.2V regulators, different package/pinout, needs a new symbol/footprint and power/clock review.

Regenerate the six sheets, netlist, BOM and previews.
Parts:
- U1: BOM Comments EOL reference baseline; footprint and operating circuit qualification pending; no LCSC listing (VIA EOL) -> EOL reference baseline; footprint and operating circuit qualification pending; no LCSC listing (VIA EOL). Non-drop-in replacement candidate: Genesys GL3510-OSY52 (LCSC C7501408), QFN-64 USB3.1 Gen1 4-port with built-in 5Vto3.3V/1.2V regulators; different package/pinout, needs a new symbol/footprint and power/clock review.
Changed lines of the file:
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@@
 (property "Manufacturer" "VIA Labs" (at 170.18 50.8 0) (effects (font (size 1 1)) hide))
 (property "Datasheet" "../../VL813.pdf" (at 170.18 50.8 0) (effects (font (size 1 1)) hide))
-(property "BOM Comments" "EOL reference baseline; footprint and operating circuit qualification pending; no LCSC listing (VIA EOL)" (at 170.18 50.8 0) (effects (font (size 1 1)) hide))
+(property "BOM Comments" "EOL reference baseline; footprint and operating circuit qualification pending; no LCSC listing (VIA EOL). Non-drop-in replacement candidate: Genesys GL3510-OSY52 (LCSC C7501408), QFN-64 USB3.1 Gen1 4-port with built-in 5Vto3.3V/1.2V regulators; different package/pinout, needs a new symbol/footprint and power/clock review." (at 170.18 50.8 0) (effects (font (size 1 1)) hide))
 (pin "23")
 (pin "22")
@@
 (property "Manufacturer" "VIA Labs" (at 254 48.26 0) (effects (font (size 1 1)) hide))
 (property "Datasheet" "../../VL813.pdf" (at 254 48.26 0) (effects (font (size 1 1)) hide))
-(property "BOM Comments" "EOL reference baseline; footprint and operating circuit qualification pending; no LCSC listing (VIA EOL)" (at 254 48.26 0) (effects (font (size 1 1)) hide))
+(property "BOM Comments" "EOL reference baseline; footprint and operating circuit qualification pending; no LCSC listing (VIA EOL). Non-drop-in replacement candidate: Genesys GL3510-OSY52 (LCSC C7501408), QFN-64 USB3.1 Gen1 4-port with built-in 5Vto3.3V/1.2V regulators; different package/pinout, needs a new symbol/footprint and power/clock review." (at 254 48.26 0) (effects (font (size 1 1)) hide))
 (pin "59")
 (pin "60")
@@
 (property "Manufacturer" "VIA Labs" (at 254 91.44 0) (effects (font (size 1 1)) hide))
 (property "Datasheet" "../../VL813.pdf" (at 254 91.44 0) (effects (font (size 1 1)) hide))
-(property "BOM Comments" "EOL reference baseline; footprint and operating circuit qualification pending; no LCSC listing (VIA EOL)" (at 254 91.44 0) (effects (font (size 1 1)) hide))
+(property "BOM Comments" "EOL reference baseline; footprint and operating circuit qualification pending; no LCSC listing (VIA EOL). Non-drop-in replacement candidate: Genesys GL3510-OSY52 (LCSC C7501408), QFN-64 USB3.1 Gen1 4-port with built-in 5Vto3.3V/1.2V regulators; different package/pinout, needs a new symbol/footprint and power/clock review." (at 254 91.44 0) (effects (font (size 1 1)) hide))
 (pin "66")
 (pin "67")
@@
 (property "Manufacturer" "VIA Labs" (at 254 134.62 0) (effects (font (size 1 1)) hide))
 (property "Datasheet" "../../VL813.pdf" (at 254 134.62 0) (effects (font (size 1 1)) hide))
-(property "BOM Comments" "EOL reference baseline; footprint and operating circuit qualification pending; no LCSC listing (VIA EOL)" (at 254 134.62 0) (effects (font (size 1 1)) hide))
+(property "BOM Comments" "EOL reference baseline; footprint and operating circuit qualification pending; no LCSC listing (VIA EOL). Non-drop-in replacement candidate: Genesys GL3510-OSY52 (LCSC C7501408), QFN-64 USB3.1 Gen1 4-port with built-in 5Vto3.3V/1.2V regulators; different package/pinout, needs a new symbol/footprint and power/clock review." (at 254 134.62 0) (effects (font (size 1 1)) hide))
 (pin "3")
 (pin "4")
@@
 (property "Manufacturer" "VIA Labs" (at 254 177.8 0) (effects (font (size 1 1)) hide))
 (property "Datasheet" "../../VL813.pdf" (at 254 177.8 0) (effects (font (size 1 1)) hide))
-(property "BOM Comments" "EOL reference baseline; footprint and operating circuit qualification pending; no LCSC listing (VIA EOL)" (at 254 177.8 0) (effects (font (size 1 1)) hide))
+(property "BOM Comments" "EOL reference baseline; footprint and operating circuit qualification pending; no LCSC listing (VIA EOL). Non-drop-in replacement candidate: Genesys GL3510-OSY52 (LCSC C7501408), QFN-64 USB3.1 Gen1 4-port with built-in 5Vto3.3V/1.2V regulators; different package/pinout, needs a new symbol/footprint and power/clock review." (at 254 177.8 0) (effects (font (size 1 1)) hide))
 (pin "11")
 (pin "12")
@@
 (property "Manufacturer" "VIA Labs" (at 294.64 243.84 0) (effects (font (size 1 1)) hide))
 (property "Datasheet" "../../VL813.pdf" (at 294.64 243.84 0) (effects (font (size 1 1)) hide))
-(property "BOM Comments" "EOL reference baseline; footprint and operating circuit qualification pending; no LCSC listing (VIA EOL)" (at 294.64 243.84 0) (effects (font (size 1 1)) hide))
+(property "BOM Comments" "EOL reference baseline; footprint and operating circuit qualification pending; no LCSC listing (VIA EOL). Non-drop-in replacement candidate: Genesys GL3510-OSY52 (LCSC C7501408), QFN-64 USB3.1 Gen1 4-port with built-in 5Vto3.3V/1.2V regulators; different package/pinout, needs a new symbol/footprint and power/clock review." (at 294.64 243.84 0) (effects (font (size 1 1)) hide))
 (pin "9")
 (pin "10")
@@
 (property "Manufacturer" "VIA Labs" (at 60.96 215.9 0) (effects (font (size 1 1)) hide))
 (property "Datasheet" "../../VL813.pdf" (at 60.96 215.9 0) (effects (font (size 1 1)) hide))
-(property "BOM Comments" "EOL reference baseline; footprint and operating circuit qualification pending; no LCSC listing (VIA EOL)" (at 60.96 215.9 0) (effects (font (size 1 1)) hide))
+(property "BOM Comments" "EOL reference baseline; footprint and operating circuit qualification pending; no LCSC listing (VIA EOL). Non-drop-in replacement candidate: Genesys GL3510-OSY52 (LCSC C7501408), QFN-64 USB3.1 Gen1 4-port with built-in 5Vto3.3V/1.2V regulators; different package/pinout, needs a new symbol/footprint and power/clock review." (at 60.96 215.9 0) (effects (font (size 1 1)) hide))
 (pin "2")
 (pin "5")
@@
 (property "Manufacturer" "VIA Labs" (at 167.64 147.32 0) (effects (font (size 1 1)) hide))
 (property "Datasheet" "../../VL813.pdf" (at 167.64 147.32 0) (effects (font (size 1 1)) hide))
-(property "BOM Comments" "EOL reference baseline; footprint and operating circuit qualification pending; no LCSC listing (VIA EOL)" (at 167.64 147.32 0) (effects (font (size 1 1)) hide))
+(property "BOM Comments" "EOL reference baseline; footprint and operating circuit qualification pending; no LCSC listing (VIA EOL). Non-drop-in replacement candidate: Genesys GL3510-OSY52 (LCSC C7501408), QFN-64 USB3.1 Gen1 4-port with built-in 5Vto3.3V/1.2V regulators; different package/pinout, needs a new symbol/footprint and power/clock review." (at 167.64 147.32 0) (effects (font (size 1 1)) hide))
 (pin "1")
 (pin "21")
